Commit message: Adding PID Control Position for Arm and Tower in RVIZ

File: siar_gazebo/models/tower_1/model.urdf (robot description, URDF)
Before this commit: robot tower, 1 links, 0 joints
Links:
- link link: geometry collision box size=4 4 10; visual mesh filename=package://siar_gazebo/models/tower_1/mesh/tower_not_3.dae

Commit message: Last SIAR version for mbzirc

File: siar_gazebo/models/tower_1/model.urdf (robot description, URDF)
Before this commit: robot tower, 1 links, 0 joints
Links:
- link link: geometry collision box size=4 4 10; visual box size=4 4 10
